Commit message: urdf: correct physical measurements to match robot
Three corrections from verified physical measurements:

1. wheel_radius: 0.033 -> 0.0325 (actual 65mm diameter / 2)
2. base_footprint -> base_link joint: use wheel_radius variable
   instead of hardcoded 0.033 so the two stay in sync
3. laser_joint X offset: 0.07 -> 0.035

The laser X offset was the largest drift: the URDF had the LiDAR
70mm ahead of base_link, but physical measurement is 35mm ahead
(chassis_centre at 65mm minus axle_offset of 30mm = 35mm).

A 35mm error in laser-to-axle offset means:
  - SLAM scans were placing obstacles 35mm closer than reality
  - DWB sim_time trajectories used wrong obstacle positions
  - Tight-corridor navigation had an asymmetric error

Physical ground-truth per earlier session:
  Chassis length: 130mm (all-in)
  Wheel diameter: 65mm -> radius 32.5mm
  Axle position: 30mm from rear, 100mm from front
  LiDAR position: 35mm ahead of axle, centre-lateral
  LiDAR height: 190mm from ground

Does NOT yet update:
  - wheel_offset_y (still 0.08, physical is 0.09 = 0.18m separation)
  - Asymmetric footprint polygon in nav2_params.yaml
These require coordinated changes with firmware WHEEL_SEPARATION_M
and navbot_base.yaml which are tracked separately in Phase C.

File: ros2_ws/src/navbot_description/urdf/navbot.urdf.xacro (robot description, xacro)
@@ -4,5 +4,5 @@
   <xacro:property name="base_width" value="0.16"/>
   <xacro:property name="base_height" value="0.06"/>
-  <xacro:property name="wheel_radius" value="0.033"/>
+  <xacro:property name="wheel_radius" value="0.0325"/>
   <xacro:property name="wheel_width" value="0.02"/>
   <xacro:property name="wheel_offset_y" value="0.08"/>
@@ -13,5 +13,5 @@
     <parent link="base_footprint"/>
     <child link="base_link"/>
-    <origin xyz="0 0 0.033" rpy="0 0 0"/>
+    <origin xyz="0 0 ${wheel_radius}" rpy="0 0 0"/>
   </joint>
   <link name="base_link">
@@ -120,5 +120,5 @@
     <parent link="base_link"/>
     <child link="laser_link"/>
-    <origin xyz="0.07 0 ${laser_height}" rpy="0 0 0"/>
+    <origin xyz="0.035 0 ${laser_height}" rpy="0 0 0"/>
   </joint>
   <link name="laser_link">
