Commit message: Phase 4: Observability and diagnostics
Firmware:
- Add DIAG command returning per-wheel PID internals:
  duty, setpoint_cps, filtered_cps, p_term, i_term, d_term, stall_timer_ms
- Add last_p_term, last_i_term, last_d_term to pid_ctrl_t for inspection
- Register NAVBOT_CMD_DIAG in protocol enum and parser

Pi serial bridge:
- Add /base/serial_latency_ms topic (PING round-trip, measured every 5s)
- Add /base/bridge_health topic (1 Hz JSON: connected, firmware version,
  uptime, reconnect count, checksum failures, odom age, latency)
- Track reconnect count and log connection number on each connect

URDF:
- Add imu_link frame as fixed joint from base_link (required by EKF
  to resolve IMU data in the robot frame)

Web console:
- Add /heading_controller/status to capture_topics default, matching
  what RUNBOOK.md documents

Tests:
- Add TestDiagnosticFields class (4 new tests) verifying PID term tracking
- Total: 81 tests passing

Co-Authored-By: Claude Opus 4.6 (1M context) <noreply@anthropic.com>

File: ros2_ws/src/navbot_description/urdf/navbot.urdf.xacro (robot description, xacro)
@@ -111,4 +111,10 @@
     </inertial>
   </link>
+  <joint name="imu_joint" type="fixed">
+    <parent link="base_link"/>
+    <child link="imu_link"/>
+    <origin xyz="0.0 0.0 ${base_height}" rpy="0 0 0"/>
+  </joint>
+  <link name="imu_link"/>
   <joint name="laser_joint" type="fixed">
     <parent link="base_link"/>

Commit message: urdf: correct wheel_offset_y to 0.091 m (empirical calibration)
2026-04-22 360° physical rotation test showed robot ~11° short of start
position. Odom reported 353.2°, physical ~349°, commanded 360°. Back-
solving: true wheel_separation = 0.180 × (353.2 / 349) ≈ 0.182 m.

Previous URDF value: wheel_offset_y = 0.08 m (separation = 0.160 m)
— 12 % smaller than physical truth. Caused TF/footprint to be
consistently narrower than reality.

New value: wheel_offset_y = 0.091 m (separation = 0.182 m) — matches
physical measurement within eyeball-level precision.

Firmware WHEEL_SEPARATION_M (0.180 m) and Pi-side odometry YAML
(0.180 m) remain unchanged. They form a self-consistent commanded-to-
odom loop; the 1.2 % deviation from physical truth is acceptable for
now and would only shift if we re-flash firmware with 0.182 and update
YAML to match. Tracked as Phase C backlog item.

Refs:
  - Rotation test data: docs/testing/motion-tests.md
  - Validation record: docs/validation/records/2026-04-22-rotation-test.md
  - Closed backlog item in docs/project-status.md
    "URDF wheel_offset_y 0.08 → 0.091 m"

Co-Authored-By: Claude Opus 4.7 (1M context) <noreply@anthropic.com>

File: ros2_ws/src/navbot_description/urdf/navbot.urdf.xacro (robot description, xacro)
@@ -6,5 +6,14 @@
   <xacro:property name="wheel_radius" value="0.0325"/>
   <xacro:property name="wheel_width" value="0.02"/>
-  <xacro:property name="wheel_offset_y" value="0.08"/>
+  <!--
+    wheel_offset_y sourced from 2026-04-22 empirical 360° rotation
+    calibration: physical ~349° vs odom 353.2° for commanded 360°
+    → true wheel_separation ≈ 0.182 m → offset = 0.091 m.
+    Prior value 0.08 was 12 % short vs truth. See
+    docs/validation/records/2026-04-22-rotation-test.md.
+    Firmware WHEEL_SEPARATION_M and Pi-side YAML wheel_separation
+    remain at 0.180 m (1.2 % low; self-consistent for odom).
+  -->
+  <xacro:property name="wheel_offset_y" value="0.091"/>
   <xacro:property name="wheel_offset_x" value="0.0"/>
   <xacro:property name="laser_height" value="0.12"/>

Commit message: imu: integrate L3G4200D + LSM303DLHC via complementary filter + EKF
End-to-end IMU integration in one session (Layers 1/2/3):

Layer 1 — IMU driver (navbot_imu/l3gd20_lsm303d_reader):
  * Added sensor_orientation param ("x_forward" | "y_forward")
    for configurable sensor→robot axis remap. New axle-height mount
    is x_forward (identity); prior chassis-top mount was y_forward.
  * Bumped poll_hz 20 → 50 Hz.
  * URDF imu_joint relocated to (0, 0, 0.035) to match axle-height
    mount.
  * Physical axis verification: tilt nose-down gave accel.x = -0.34 g,
    accel.y ≈ 0 (X-forward confirmed). 90° CCW rotation gave
    quaternion.z = +0.667 → +83° (right-hand-rule confirmed).

Layer 2 — imu_complementary_filter:
  * New imu_fusion.launch.py remaps driver output to the standard
    /imu/data_raw + /imu/mag topics and launches the complementary
    filter with use_mag: false.
  * Magnetometer deferred — field magnitude at axle-height mount
    is 1.43 gauss, ~2.3× Earth's max. Strong hard-iron bias from
    motor magnets. Calibration pass logged as backlog item.

Layer 3 — robot_localization EKF:
  * Rewrote ekf.yaml: wheel odom contributes x, y, vx; IMU (fused
    /imu/data) contributes yaw, vyaw. 2D mode. 30 Hz output on
    /odometry/filtered.
  * EKF now owns odom → base_footprint TF. Flipped
    navbot_serial_bridge.publish_tf: true → false.
  * Fixed launch-time bug: ekf.launch.py was passing
    {"use_sim_time": LaunchConfiguration(...)} which resolves to a
    STRING that robot_localization treats as truthy, causing the
    node to block on "Waiting for clock to start...". Removed the
    launch override; use_sim_time comes from yaml.

Nav2 switched odom_topic: /odom → /odometry/filtered (bt_navigator
and velocity_smoother).

Top-level slam_imu.launch.py brings up base + LiDAR + SLAM + IMU
fusion + EKF in one shot.

End-to-end validation — 180° in-place rotation:
  Pre-EKF (pre-damping, session 8): 95° overshoot + oscillation
  Pre-EKF (post-damping, session 9 A): 13° error + one reversal
  Post-EKF (this commit):  clean monotonic sweep at -0.287 ±
    0.013 rad/s across 108 samples, no reversals, 12.4° terminal
    error (goal-checker settling delay).

Also opens backlog items: mag-cal, navbot_base.yaml wheel_radius
alignment, pre-EKF base bring-up mode.

Co-Authored-By: Claude Opus 4.7 (1M context) <noreply@anthropic.com>

File: ros2_ws/src/navbot_description/urdf/navbot.urdf.xacro (robot description, xacro)
@@ -123,5 +123,11 @@
     <parent link="base_link"/>
     <child link="imu_link"/>
-    <origin xyz="0.0 0.0 ${base_height}" rpy="0 0 0"/>
+    <!-- 2026-04-22 (session 9): IMU relocated from chassis top
+         (base_height = 0.06) to axle height (0.035 m). Closer to the
+         center of rotation reduces centripetal-acceleration cross-
+         coupling during turns. Phase 0 post-move: accel Z = +0.9 g
+         (Z-up confirmed); mag magnitude 1.43 gauss (strong local
+         source from motors — mag deferred to backlog). -->
+    <origin xyz="0.0 0.0 0.035" rpy="0 0 0"/>
   </joint>
   <link name="imu_link"/>
